File: MFOS Dual VCA 2Layer.brd (EAGLE design)
At the start: 98.7 x 80 mm, 61 parts, among them IC1 TL072P, IC2 LM13700N, Q1 2N3904, Q2 2N3904, Q3 2N3906, Q4 2N3906, U1 POWER

Commit message: routed and doing labels
Parts:
- removed TRIM_A1, TRIM_A2: 2k, pot:B64W
- added TRIM1, TRIM2: (no value), pot:S64YW
- BIAS1, BIAS2: value 100k -> (none); device pot:B64W -> pot:S64YW
- R1, R10, R11, R12, R13, R14, R15, R16, R17, R18, R19, R2, R20, R21, R22, R23, R24, R25, R26, R27, R28, R3, R4, R5, R6, R7, R8, R9: device rcl:R1206 -> rcl:0207/7
- moved Q4 155.8 mm to (76.2, 31.8), turned to 180 degrees
- moved R15 154.2 mm to (67.3, 24.1), turned to 270 degrees
- moved R12 148.8 mm to (76.2, 39.4), turned to 270 degrees
- moved R14 147.0 mm to (64.8, 24.1), turned to 90 degrees
- moved R5 143.8 mm to (69.8, 24.1), turned to 270 degrees
- moved CMNA1 136.8 mm to (81.3, 34.3)
- moved BIAS1 136.0 mm to (52.1, 22.9), turned to 90 degrees
- moved R20 135.3 mm to (54.6, 44.5), turned to 270 degrees
- moved Q3 134.7 mm to (71.1, 41.9)
- moved R17 122.2 mm to (27.9, 24.1), turned to 90 degrees
- moved R8 121.5 mm to (39.4, 44.5), turned to 270 degrees
- moved R13 119.8 mm to (77.5, 19.1)
- moved ADJ1 119.1 mm to (36.8, 15.2)
- moved Q2 117.7 mm to (71.1, 38.1), turned to 180 degrees
- moved IC2 117.0 mm to (55.9, 34.3)
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- renumbered 1N1 to IN1
Connections:
- net +12V: now also BIAS1.E, BIAS2.E; no longer BIAS1.A, BIAS2.A
- net -12V: now also BIAS1.A, BIAS2.A; no longer BIAS1.E, BIAS2.E
- net N$18: no longer BIAS1.P$1
- net N$22: now also TRIM1.A; no longer TRIM_A1.E
- net N$23: now also TRIM1.E, TRIM1.S; no longer TRIM_A1.A, TRIM_A1.P$1, TRIM_A1.S
- net N$28: no longer BIAS2.P$1
- net N$29: now also TRIM2.A; no longer TRIM_A2.E
- net N$30: now also TRIM2.E, TRIM2.S; no longer TRIM_A2.A, TRIM_A2.P$1, TRIM_A2.S
Routing:
- net GND: track 0.00 -> 282.0 mm
- net +12V: track 0.00 -> 208.2 mm
- net -12V: track 0.00 -> 190.9 mm
- net N$25: track 0.00 -> 126.2 mm, vias 0 -> 1
- net N$1: track 0.00 -> 90.7 mm
- net N$9: track 0.00 -> 83.0 mm
- net N$5: track 0.00 -> 66.4 mm
- net N$8: track 0.00 -> 56.8 mm
- net N$17: track 0.00 -> 48.1 mm, vias 0 -> 1
- net N$3: track 0.00 -> 42.3 mm
- net N$15: track 0.00 -> 41.6 mm, vias 0 -> 2
- net N$23: track 0.00 -> 40.6 mm, vias 0 -> 1
- net N$16: track 0.00 -> 36.9 mm
- net N$11: track 0.00 -> 35.8 mm
- net N$22: track 0.00 -> 32.7 mm
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Other:
- board size 98.7 x 80 mm -> 98.7 x 57.1 mm
